File: PCB/stm32-module.kicad_pcb (KiCad board)
At the start: 4 copper layers, 45.5 x 78.5 mm, 35 parts, among them J1 Conn_01x30_Socket, J2 Conn_01x30_Socket, J3 TYPE-C_16PIN_2MD__073_

Commit message: changed images to reflect changes
Parts:
- J1, J2: footprint Connector_PinSocket_2.54mm:PinSocket_1x30_P2.54mm_Vertical -> Connector_PinHeader_2.54mm:PinHeader_1x30_P2.54mm_Vertical
Changed lines of the file:
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@@
 		(model "${EASYEDA2KICAD}/easyeda2kicad.3dshapes/SOT-223-4P_L6.5-W3.5-H1.6-LS7.0-P2.30.wrl"
 			(offset
-				(xyz -3.99 2.92 -0)
+				(xyz 0 0 -0)
 			)
 			(scale
@@
 			)
 			(rotate
-				(xyz 0 0 180)
+				(xyz -0 -0 180)
 			)
 		)
@@
 		)
 	)
-	(footprint "Connector_PinSocket_2.54mm:PinSocket_1x30_P2.54mm_Vertical"
+	(footprint "Connector_PinHeader_2.54mm:PinHeader_1x30_P2.54mm_Vertical"
 		(layer "F.Cu")
 		(at 83.7 40.21)
-		(descr "Through hole straight socket strip, 1x30, 2.54mm pitch, single row (from Kicad 4.0.7), script generated")
-		(tags "Through hole socket strip THT 1x30 2.54mm single row")
+		(descr "Through hole straight pin header, 1x30, 2.54mm pitch, single row")
+		(tags "Through hole pin header THT 1x30 2.54mm single row")
 		(property "Reference" "J1"
-			(at 0 -2.77 0)
+			(at 0 -2.38 0)
 			(layer "F.SilkS")
-			(hide yes)
 			(effects
 				(font
@@
 		)
 		(property "Value" "Conn_01x30_Socket"
-			(at 0 76.43 0)
+			(at 0 76.04 0)
 			(layer "F.Fab")
-			(hide yes)
 			(effects
 				(font
@@
 			)
 		)
-		(property "Description" "Generic connector, single row, 01x30, script generated"
+		(property "Description" ""
 			(at 0 0 0)
 			(layer "F.Fab")
@@
 		(sheetname "/")
 		(sheetfile "stm32-module.kicad_sch")
-		(units
-			(unit
-				(name "A")
-				(pins "1" "2" "3" "4" "5" "6" "7" "8" "9" "10" "11" "12" "13" "14" "15"
-					"16" "17" "18" "19" "20" "21" "22" "23" "24" "25" "26" "27" "28" "29"
-					"30"
-				)
-			)
-		)
 		(attr through_hole)
 		(duplicate_pad_numbers_are_jumpers no)
 		(fp_line
-			(start -1.33 1.27)
-			(end -1.33 74.99)
+			(start -1.38 -1.38)
+			(end 0 -1.38)
 			(stroke
 				(width 0.12)
@@
 		)
 		(fp_line
-			(start -1.33 1.27)
-			(end 1.33 1.27)
+			(start -1.38 0)
+			(end -1.38 -1.38)
 			(stroke
 				(width 0.12)
@@
 		)
 		(fp_line
-			(start -1.33 74.99)
-			(end 1.33 74.99)
+			(start -1.38 1.27)
+			(end -1.38 75.04)
 			(stroke
 				(width 0.12)
@@
 		)
 		(fp_line
-			(start 0 -1.33)
-			(end 1.33 -1.33)
+			(start -1.38 1.27)
+			(end 1.38 1.27)
 			(stroke
 				(width 0.12)
@@
 		)
 		(fp_line
-			(start 1.33 -1.33)
-			(end 1.33 0)
+			(start -1.38 75.04)
+			(end 1.38 75.04)
 			(stroke
 				(width 0.12)
@@
 		)
 		(fp_line
-			(start 1.33 1.27)
-			(end 1.33 74.99)
+			(start 1.38 1.27)
+			(end 1.38 75.04)
 			(stroke
 				(width 0.12)
@@
 			(layer "F.SilkS")
 		)
-		(fp_line
+		(fp_rect
 			(start -1.77 -1.77)
-			(end 1.77 -1.77)
-			(stroke
-				(width 0.05)
-				(type solid)
-			)
-			(layer "F.CrtYd")
-		)
-		(fp_line
-			(start -1.77 75.43)
-			(end -1.77 -1.77)
-			(stroke
-				(width 0.05)
-				(type solid)
-			)
-			(layer "F.CrtYd")
-		)
-		(fp_line
-			(start 1.77 -1.77)
 			(end 1.77 75.43)
 			(stroke
@@
 				(type solid)
 			)
+			(fill no)
 			(layer "F.CrtYd")
 		)
 		(fp_line
-			(start 1.77 75.43)
-			(end -1.77 75.43)
-			(stroke
-				(width 0.05)
-				(type solid)
-			)
-			(layer "F.CrtYd")
-		)
-		(fp_line
-			(start -1.27 -1.27)
-			(end 0.635 -1.27)
+			(start -1.27 -0.635)
+			(end -0.635 -1.27)
 			(stroke
 				(width 0.1)
@@
 		(fp_line
 			(start -1.27 74.93)
-			(end -1.27 -1.27)
+			(end -1.27 -0.635)
 			(stroke
 				(width 0.1)
@@
 		)
 		(fp_line
-			(start 0.635 -1.27)
-			(end 1.27 -0.635)
+			(start -0.635 -1.27)
+			(end 1.27 -1.27)
 			(stroke
 				(width 0.1)
@@
 		)
 		(fp_line
-			(start 1.27 -0.635)
+			(start 1.27 -1.27)
 			(end 1.27 74.93)
 			(stroke
@@
 		)
 		(embedded_fonts no)
-		(model "${KICAD10_3DMODEL_DIR}/Connector_PinSocket_2.54mm.3dshapes/PinSocket_1x30_P2.54mm_Vertical.step"
+		(model "${KICAD10_3DMODEL_DIR}/Connector_PinHeader_2.54mm.3dshapes/PinHeader_1x30_P2.54mm_Vertical.step"
 			(offset
 				(xyz 0 0 0)
@@
 		)
 		(embedded_fonts no)
-		(model "C:\\Users\\ember\\Documents\\KiCad\\8.0\\cse\\SamacSys_Parts.3dshapes\\TPS73618QDCQRQ1.stp"
+		(model "/home/ember/Downloads/DCQ0006A.stp"
 			(offset
 				(xyz 0 0 0)
@@
 		)
 		(embedded_fonts no)
-		(model "C:\\Users\\ember\\Documents\\KiCad\\8.0\\cse\\SamacSys_Parts.3dshapes\\STM32H7B0RBT6.stp"
+		(model "${EASYEDA2KICAD}/easyeda2kicad.3dshapes/LQFP-64_L10.0-W10.0-H1.4-LS12.0-P0.50.step"
 			(offset
-				(xyz 1.789999935 -8.770000326 0.9599999641)
+				(xyz 0 0 0)
 			)
 			(scale
@@
 			)
 			(rotate
-				(xyz 0 0 0)
+				(xyz -0 -0 90)
 			)
 		)
@@
 		)
 	)
-	(footprint "Connector_PinSocket_2.54mm:PinSocket_1x30_P2.54mm_Vertical"
+	(footprint "Connector_PinHeader_2.54mm:PinHeader_1x30_P2.54mm_Vertical"
 		(layer "F.Cu")
 		(at 124.46 40.21)
-		(descr "Through hole straight socket strip, 1x30, 2.54mm pitch, single row (from Kicad 4.0.7), script generated")
-		(tags "Through hole socket strip THT 1x30 2.54mm single row")
+		(descr "Through hole straight pin header, 1x30, 2.54mm pitch, single row")
+		(tags "Through hole pin header THT 1x30 2.54mm single row")
 		(property "Reference" "J2"
-			(at 0 -2.77 0)
+			(at 0 -2.38 0)
 			(layer "F.SilkS")
-			(hide yes)
 			(effects
 				(font
@@
 		)
 		(property "Value" "Conn_01x30_Socket"
-			(at 0 76.43 0)
+			(at 0 76.04 0)
 			(layer "F.Fab")
-			(hide yes)
 			(effects
 				(font
@@
 			)
 		)
-		(property "Description" "Generic connector, single row, 01x30, script generated"
+		(property "Description" ""
 			(at 0 0 0)
 			(layer "F.Fab")
@@
 		(sheetname "/")
 		(sheetfile "stm32-module.kicad_sch")
-		(units
-			(unit
-				(name "A")
-				(pins "1" "2" "3" "4" "5" "6" "7" "8" "9" "10" "11" "12" "13" "14" "15"
-					"16" "17" "18" "19" "20" "21" "22" "23" "24" "25" "26" "27" "28" "29"
-					"30"
-				)
-			)
-		)
 		(attr through_hole)
 		(duplicate_pad_numbers_are_jumpers no)
 		(fp_line
-			(start -1.33 1.27)
-			(end -1.33 74.99)
+			(start -1.38 -1.38)
+			(end 0 -1.38)
 			(stroke
 				(width 0.12)
@@
 		)
 		(fp_line
-			(start -1.33 1.27)
-			(end 1.33 1.27)
+			(start -1.38 0)
+			(end -1.38 -1.38)
 			(stroke
 				(width 0.12)
@@
 		)
 		(fp_line
-			(start -1.33 74.99)
-			(end 1.33 74.99)
+			(start -1.38 1.27)
+			(end -1.38 75.04)
 			(stroke
 				(width 0.12)
@@
 		)
 		(fp_line
-			(start 0 -1.33)
-			(end 1.33 -1.33)
+			(start -1.38 1.27)
+			(end 1.38 1.27)
 			(stroke
 				(width 0.12)
@@
 		)
 		(fp_line
-			(start 1.33 -1.33)
-			(end 1.33 0)
+			(start -1.38 75.04)
+			(end 1.38 75.04)
 			(stroke
 				(width 0.12)
@@
 		)
 		(fp_line
-			(start 1.33 1.27)
-			(end 1.33 74.99)
+			(start 1.38 1.27)
+			(end 1.38 75.04)
 			(stroke
 				(width 0.12)
@@
 			(layer "F.SilkS")
 		)
-		(fp_line
+		(fp_rect
 			(start -1.77 -1.77)
-			(end 1.77 -1.77)
-			(stroke
-				(width 0.05)
-				(type solid)
-			)
-			(layer "F.CrtYd")
-		)
-		(fp_line
-			(start -1.77 75.43)
-			(end -1.77 -1.77)
-			(stroke
-				(width 0.05)
-				(type solid)
-			)
-			(layer "F.CrtYd")
-		)
-		(fp_line
-			(start 1.77 -1.77)
 			(end 1.77 75.43)
 			(stroke
@@
 				(type solid)
 			)
+			(fill no)
 			(layer "F.CrtYd")
 		)
 		(fp_line
-			(start 1.77 75.43)
-			(end -1.77 75.43)
-			(stroke
-				(width 0.05)
-				(type solid)
-			)
-			(layer "F.CrtYd")
-		)
-		(fp_line
-			(start -1.27 -1.27)
-			(end 0.635 -1.27)
+			(start -1.27 -0.635)
+			(end -0.635 -1.27)
 			(stroke
 				(width 0.1)
@@
 		(fp_line
 			(start -1.27 74.93)
-			(end -1.27 -1.27)
+			(end -1.27 -0.635)
 			(stroke
 				(width 0.1)
@@
 		)
 		(fp_line
-			(start 0.635 -1.27)
-			(end 1.27 -0.635)
+			(start -0.635 -1.27)
+			(end 1.27 -1.27)
 			(stroke
 				(width 0.1)
@@
 		)
 		(fp_line
-			(start 1.27 -0.635)
+			(start 1.27 -1.27)
 			(end 1.27 74.93)
 			(stroke
@@
 		)
 		(embedded_fonts no)
-		(model "${KICAD10_3DMODEL_DIR}/Connector_PinSocket_2.54mm.3dshapes/PinSocket_1x30_P2.54mm_Vertical.step"
+		(model "${KICAD10_3DMODEL_DIR}/Connector_PinHeader_2.54mm.3dshapes/PinHeader_1x30_P2.54mm_Vertical.step"
 			(offset
 				(xyz 0 0 0)
